File: pcb/pisces/pisces.kicad_pcb (KiCad board)
At the start: 2 copper layers, 149.9 x 66 mm, 51 parts, among them SW1 SW_PUSH, SW10 SW_PUSH, SW11 SW_PUSH, SW12 SW_PUSH, SW13 SW_PUSH, SW14 SW_PUSH, SW15 SW_PUSH, SW16 SW_PUSH, SW17 SW_PUSH, SW18 SW_PUSH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

Commit message: Issue3 add jack (#4)
* Added a audio jack and connected tracks

* Filled GND area

* Aligned mounting holes
Parts:
- added J1: AudioJack4, Connector_Audio:Jack_3.5mm_PJ320D_Horizontal, F.Cu at (187.2, 44.6)
- moved Ref** 14.8 mm to (189.1, 54.9)
- moved Ref** 4.07 mm to (189.1, 72.6)
- moved Ref** 2.92 mm to (159.6, 43.6)
Connections:
- U1 pad 2: Net-(U1-Pad2) -> data
Routing:
- net data: track 0.00 -> 28.9 mm
- net GND: track 60.8 -> 72.2 mm
- net VCC: track 33.4 -> 44.3 mm, vias 0 -> 1
- net col4: track 206.2 -> 205.3 mm
- net col5: track 191.9 -> 191.0 mm
- net col3: track 224.2 -> 223.3 mm
- net col2: track 240.8 -> 240.0 mm
- net col1: track 258.3 -> 257.5 mm
- net col0: track 274.4 -> 273.6 mm
- added copper zone on B.Cu, net GND
- added copper zone on F.Cu, net GND
Other:
- board size 149.9 x 66 mm -> 154.9 x 66 mm

Commit message: Updated foot prints to reversible
Routing:
- net VCC: track 44.3 -> 57.9 mm, vias 1 -> 2
- net GND: track 72.2 -> 83.5 mm, vias 0 -> 1
- net Net-(J1-PadS): track 0.00 -> 6.49 mm, vias 0 -> 1
- net Net-(LED1-Pad2): track 0.00 -> 6.23 mm, vias 0 -> 1
- net led: track 36.1 -> 42.1 mm
- net reset: track 30.5 -> 33.3 mm, vias 0 -> 1
- net data: track 28.9 -> 31.2 mm, vias 0 -> 1

Commit message: Added pisces bottom plate (#8)
Parts:
- renumbered Ref** to hh1, Ref** to hh2, Ref** to hh3, Ref** to hh4
