File: pcb/v2/pisces_bottom_plate.kicad_pcb (KiCad board)
At the start: 2 copper layers, 154.9 x 66 mm, 10 parts

Commit message: bottom plate is done
Parts:
- removed ? (x10): , kbd:M2_Hole_TH
- added REF**: M2_Hole_TH, kbd:M2_Hole_TH, F.Cu at (59.5, 59.5)
- added REF**: M2_Hole_TH, kbd:M2_Hole_TH, F.Cu at (135.7, 78.6)
- added REF**: M2_Hole_TH, kbd:M2_Hole_TH, F.Cu at (135.7, 59.5)
- added REF**: M2_Hole_TH, kbd:M2_Hole_TH, F.Cu at (97.6, 78.6)
- added REF**: M2_Hole_TH, kbd:M2_Hole_TH, F.Cu at (97.6, 59.5)
- added REF**: M2_Hole_TH, kbd:M2_Hole_TH, F.Cu at (59.5, 78.6)
Other:
- board size 154.9 x 66 mm -> 137.8 x 60.1 mm
Changed lines of the file:
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@@
   (general
     (thickness 1.6)
-    (drawings 8)
-    (tracks 1)
+    (drawings 16)
+    (tracks 0)
     (zones 0)
-    (modules 10)
+    (modules 6)
     (nets 1)
   )
@@
       (drillshape 0)
       (scaleselection 1)
-      (outputdirectory "gerber/bottom_plate/"))
+      (outputdirectory "gerber/pcb/"))
   )
   (net 0 "")
@@
   )
   (module kbd:M2_Hole_TH (layer F.Cu)
-    (at 59.525 78.575)
-    (fp_text reference "" (at 0 0.5) (layer F.SilkS) hide
+    (at 59.525 59.525)
+    (fp_text reference REF** (at 0 0.5) (layer F.SilkS)
       (effects (font (size 1 1) (thickness 0.15)))
     )
-    (fp_text value "" (at 0 -0.5) (layer F.Fab) hide
+    (fp_text value M2_Hole_TH (at 0 -0.5) (layer F.Fab)
       (effects (font (size 1 1) (thickness 0.15)))
     )
@@
   )
   (module kbd:M2_Hole_TH (layer F.Cu)
-    (at 159.639 43.561)
-    (fp_text reference "" (at 0 0.5) (layer F.SilkS) hide
+    (at 135.725 78.575)
+    (fp_text reference REF** (at 0 0.5) (layer F.SilkS)
       (effects (font (size 1 1) (thickness 0.15)))
     )
-    (fp_text value "" (at 0 -0.5) (layer F.Fab) hide
+    (fp_text value M2_Hole_TH (at 0 -0.5) (layer F.Fab)
       (effects (font (size 1 1) (thickness 0.15)))
     )
@@
   (module kbd:M2_Hole_TH (layer F.Cu)
     (at 135.725 59.525)
-    (fp_text reference "" (at 0 0.5) (layer F.SilkS) hide
+    (fp_text reference REF** (at 0 0.5) (layer F.SilkS)
       (effects (font (size 1 1) (thickness 0.15)))
     )
-    (fp_text value "" (at 0 -0.5) (layer F.Fab) hide
-      (effects (font (size 1 1) (thickness 0.15)))
-    )
-    (pad "" thru_hole circle (at 0 0) (size 4.2 4.2) (drill 2.3) (layers *.Cu *.Mask))
-  )
-  (module kbd:M2_Hole_TH (layer F.Cu)
-    (at 135.725 78.575)
-    (fp_text reference "" (at 0 0.5) (layer F.SilkS) hide
-      (effects (font (size 1 1) (thickness 0.15)))
-    )
-    (fp_text value "" (at 0 -0.5) (layer F.Fab) hide
+    (fp_text value M2_Hole_TH (at 0 -0.5) (layer F.Fab)
       (effects (font (size 1 1) (thickness 0.15)))
     )
@@
   (module kbd:M2_Hole_TH (layer F.Cu)
     (at 97.625 78.575)
-    (fp_text reference "" (at 0 0.5) (layer F.SilkS) hide
+    (fp_text reference REF** (at 0 0.5) (layer F.SilkS)
       (effects (font (size 1 1) (thickness 0.15)))
     )
-    (fp_text value "" (at 0 -0.5) (layer F.Fab) hide
-      (effects (font (size 1 1) (thickness 0.15)))
-    )
-    (pad "" thru_hole circle (at 0 0) (size 4.2 4.2) (drill 2.3) (layers *.Cu *.Mask))
-  )
-  (module kbd:M2_Hole_TH (layer F.Cu)
-    (at 189.103 72.644)
-    (fp_text reference "" (at 0 0.5) (layer F.SilkS) hide
-      (effects (font (size 1 1) (thickness 0.15)))
-    )
-    (fp_text value "" (at 0 -0.5) (layer F.Fab) hide
-      (effects (font (size 1 1) (thickness 0.15)))
-    )
-    (pad "" thru_hole circle (at 0 0) (size 4.2 4.2) (drill 2.3) (layers *.Cu *.Mask))
-  )
-  (module kbd:M2_Hole_TH (layer F.Cu)
-    (at 189.103 54.864)
-    (fp_text reference "" (at 0 0.5) (layer F.SilkS) hide
-      (effects (font (size 1 1) (thickness 0.15)))
-    )
-    (fp_text value "" (at 0 -0.5) (layer F.Fab) hide
-      (effects (font (size 1 1) (thickness 0.15)))
-    )
-    (pad "" thru_hole circle (at 0 0) (size 4.2 4.2) (drill 2.3) (layers *.Cu *.Mask))
-  )
-  (module kbd:M2_Hole_TH (layer F.Cu)
-    (at 159.639 72.644)
-    (fp_text reference "" (at 0 0.5) (layer F.SilkS) hide
-      (effects (font (size 1 1) (thickness 0.15)))
-    )
-    (fp_text value "" (at 0 -0.5) (layer F.Fab) hide
+    (fp_text value M2_Hole_TH (at 0 -0.5) (layer F.Fab)
       (effects (font (size 1 1) (thickness 0.15)))
     )
@@
   (module kbd:M2_Hole_TH (layer F.Cu)
     (at 97.625 59.525)
-    (fp_text reference "" (at 0 0.5) (layer F.SilkS) hide
+    (fp_text reference REF** (at 0 0.5) (layer F.SilkS)
       (effects (font (size 1 1) (thickness 0.15)))
     )
-    (fp_text value "" (at 0 -0.5) (layer F.Fab) hide
+    (fp_text value M2_Hole_TH (at 0 -0.5) (layer F.Fab)
       (effects (font (size 1 1) (thickness 0.15)))
     )
@@
   )
   (module kbd:M2_Hole_TH (layer F.Cu)
-    (at 59.525 59.525)
-    (fp_text reference "" (at 0 0.5) (layer F.SilkS) hide
+    (at 59.525 78.575)
+    (fp_text reference REF** (at 0 0.5) (layer F.SilkS)
       (effects (font (size 1 1) (thickness 0.15)))
     )
-    (fp_text value "" (at 0 -0.5) (layer F.Fab) hide
+    (fp_text value M2_Hole_TH (at 0 -0.5) (layer F.Fab)
       (effects (font (size 1 1) (thickness 0.15)))
     )
     (pad "" thru_hole circle (at 0 0) (size 4.2 4.2) (drill 2.3) (layers *.Cu *.Mask))
   )
-  (gr_arc (start 189.23 38.1) (end 193.04 38.1) (angle -90) (layer Edge.Cuts) (width 0.05))
-  (gr_arc (start 41.91 38.1) (end 41.91 34.29) (angle -90) (layer Edge.Cuts) (width 0.05))
-  (gr_arc (start 189.23 96.52) (end 189.23 100.33) (angle -90) (layer Edge.Cuts) (width 0.05))
-  (gr_arc (start 41.91 96.52) (end 38.1 96.52) (angle -90) (layer Edge.Cuts) (width 0.05))
-  (gr_line (start 189.23 34.29) (end 41.91 34.29) (layer Edge.Cuts) (width 0.05))
-  (gr_line (start 193.04 96.52) (end 193.04 38.1) (layer Edge.Cuts) (width 0.05))
-  (gr_line (start 41.91 100.33) (end 189.23 100.33) (layer Edge.Cuts) (width 0.05))
-  (gr_line (start 38.1 38.1) (end 38.1 96.52) (layer Edge.Cuts) (width 0.05))
-  (segment (start 135.814 59.436) (end 135.725 59.525) (width 0.25) (layer B.Cu) (net 0))
+  (gr_line (start 157.48 44.45) (end 163.576 44.45) (layer Edge.Cuts) (width 0.05))
+  (gr_line (start 164.846 40.259) (end 164.846 43.18) (layer Edge.Cuts) (width 0.05))
+  (gr_line (start 156.21 40.259) (end 156.21 43.18) (layer Edge.Cuts) (width 0.05))
+  (gr_arc (start 166.116 40.259) (end 166.116 38.989) (angle -90) (layer Edge.Cuts) (width 0.05))
+  (gr_arc (start 163.576 43.18) (end 163.576 44.45) (angle -90) (layer Edge.Cuts) (width 0.05))
+  (gr_arc (start 157.48 43.18) (end 156.21 43.18) (angle -90) (layer Edge.Cuts) (width 0.05))
+  (gr_arc (start 154.94 40.259) (end 156.21 40.259) (angle -90) (layer Edge.Cuts) (width 0.05))
+  (gr_arc (start 174.244 41.529) (end 176.784 41.529) (angle -90) (layer Edge.Cuts) (width 0.05))
+  (gr_arc (start 174.244 96.52) (end 174.244 99.06) (angle -90) (layer Edge.Cuts) (width 0.05))
+  (gr_arc (start 41.529 96.52) (end 38.989 96.52) (angle -90) (layer Edge.Cuts) (width 0.05))
+  (gr_arc (start 41.529 41.529) (end 41.529 38.989) (angle -90) (layer Edge.Cuts) (width 0.05))
+  (gr_line (start 174.244 38.989) (end 166.116 38.989) (layer Edge.Cuts) (width 0.05))
+  (gr_line (start 154.94 38.989) (end 41.529 38.989) (layer Edge.Cuts) (width 0.05))
+  (gr_line (start 176.784 96.52) (end 176.784 41.529) (layer Edge.Cuts) (width 0.05))
+  (gr_line (start 41.529 99.06) (end 174.244 99.06) (layer Edge.Cuts) (width 0.05))
+  (gr_line (start 38.989 41.529) (end 38.989 96.52) (layer Edge.Cuts) (width 0.05))
   (zone (net 0) (net_name "") (layer F.Cu) (hatch edge 0.508)
     (connect_pads (clearance 0.508))
@@
     (polygon
       (pts
-        (xy 193.04 100.33) (xy 38.1 100.33) (xy 38.1 34.29) (xy 193.04 34.29)
+        (xy 177.8 101.6) (xy 38.1 101.6) (xy 38.1 38.1) (xy 177.8 38.1)
       )
     )
@@
     (polygon
       (pts
-        (xy 193.04 100.33) (xy 38.1 100.33) (xy 38.1 34.29) (xy 193.04 34.29)
+        (xy 177.8 101.6) (xy 38.1 101.6) (xy 38.1 38.1) (xy 177.8 38.1)
       )
     )
