File: pcb/v2/pisces_top_plate.kicad_pcb (KiCad board)
At the start: 2 copper layers, 137.2 x 66 mm, 6 parts

Commit message: done with top plate
Parts:
- removed ? (x6): , kbd:M2_Hole_TH
- added REF**: M2_Hole_TH, kbd:M2_Hole_TH, F.Cu at (135.7, 78.6)
- added REF**: M2_Hole_TH, kbd:M2_Hole_TH, F.Cu at (97.6, 78.6)
- added REF**: M2_Hole_TH, kbd:M2_Hole_TH, F.Cu at (135.7, 59.5)
- added REF**: M2_Hole_TH, kbd:M2_Hole_TH, F.Cu at (97.6, 59.5)
- added REF**: M2_Hole_TH, kbd:M2_Hole_TH, F.Cu at (59.5, 78.6)
- added REF**: M2_Hole_TH, kbd:M2_Hole_TH, F.Cu at (59.5, 59.5)
Other:
- board size 137.2 x 66 mm -> 137.8 x 60.1 mm
