File: pcb/v2/pisces.sch (KiCad schematic (older format))
At the start: 55 parts, among them J1 USB_B_Micro, J2 AudioJack4, SW1 SW_PUSH, SW10 SW_PUSH, SW11 SW_PUSH, SW12 SW_PUSH, SW13 SW_PUSH, SW14 SW_PUSH, SW15 SW_PUSH, SW16 SW_PUSH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

Commit message: Resistors: 0805 --> 0603, Capacitors (other than 10u): 0603
Parts:
- R1, R2, R3, R4: footprint Resistor_SMD:R_0805_2012Metric -> Resistor_SMD:R_0603_1608Metric
Changed lines of the file:
@@
 F 0 "R1" V 1293 6200 50  0000 C CNN
 F 1 "22" V 1384 6200 50  0000 C CNN
-F 2 "Resistor_SMD:R_0805_2012Metric" V 1430 6200 50  0001 C CNN
+F 2 "Resistor_SMD:R_0603_1608Metric" V 1430 6200 50  0001 C CNN
 F 3 "~" H 1500 6200 50  0001 C CNN
 	1    1500 6200
@@
 F 0 "R2" V 1543 6300 50  0000 C CNN
 F 1 "22" V 1634 6300 50  0000 C CNN
-F 2 "Resistor_SMD:R_0805_2012Metric" V 1680 6300 50  0001 C CNN
+F 2 "Resistor_SMD:R_0603_1608Metric" V 1680 6300 50  0001 C CNN
 F 3 "~" H 1750 6300 50  0001 C CNN
 	1    1750 6300
@@
 F 0 "R3" H 4645 3921 50  0000 L CNN
 F 1 "10k" H 4645 3830 50  0000 L CNN
-F 2 "Resistor_SMD:R_0805_2012Metric" V 4505 3875 50  0001 C CNN
+F 2 "Resistor_SMD:R_0603_1608Metric" V 4505 3875 50  0001 C CNN
 F 3 "~" H 4575 3875 50  0001 C CNN
 	1    4575 3875
@@
 F 0 "R4" H 6259 6546 50  0000 L CNN
 F 1 "10k" H 6259 6455 50  0000 L CNN
-F 2 "Resistor_SMD:R_0805_2012Metric" H 6200 6500 50  0001 C CNN
+F 2 "Resistor_SMD:R_0603_1608Metric" H 6200 6500 50  0001 C CNN
 F 3 "~" H 6200 6500 50  0001 C CNN
 	1    6200 6500

Commit message: Smaller parts footprint
Parts:
- C1, C2, C3, C6: footprint Capacitor_SMD:C_0603_1608Metric -> Capacitor_SMD:C_0402_1005Metric
Changed lines of the file:
@@
 F 0 "C3" H 4715 5221 50  0000 L CNN
 F 1 "0.1u" H 4715 5130 50  0000 L CNN
-F 2 "Capacitor_SMD:C_0603_1608Metric" H 4638 5025 50  0001 C CNN
+F 2 "Capacitor_SMD:C_0402_1005Metric" H 4638 5025 50  0001 C CNN
 F 3 "~" H 4600 5175 50  0001 C CNN
 	1    4600 5175
@@
 F 0 "C1" H 3692 4496 50  0000 L CNN
 F 1 "22p" H 3692 4405 50  0000 L CNN
-F 2 "Capacitor_SMD:C_0603_1608Metric" H 3600 4450 50  0001 C CNN
+F 2 "Capacitor_SMD:C_0402_1005Metric" H 3600 4450 50  0001 C CNN
 F 3 "~" H 3600 4450 50  0001 C CNN
 	1    3600 4450
@@
 F 0 "C2" H 3867 4671 50  0000 L CNN
 F 1 "22p" H 3867 4580 50  0000 L CNN
-F 2 "Capacitor_SMD:C_0603_1608Metric" H 3775 4625 50  0001 C CNN
+F 2 "Capacitor_SMD:C_0402_1005Metric" H 3775 4625 50  0001 C CNN
 F 3 "~" H 3775 4625 50  0001 C CNN
 	1    3775 4625
@@
 F 0 "C6" H 3192 6146 50  0000 L CNN
 F 1 "0.1u" H 3192 6055 50  0000 L CNN
-F 2 "Capacitor_SMD:C_0603_1608Metric" H 3100 6100 50  0001 C CNN
+F 2 "Capacitor_SMD:C_0402_1005Metric" H 3100 6100 50  0001 C CNN
 F 3 "~" H 3100 6100 50  0001 C CNN
 	1    3100 6100
