File: pcb/v2/pisces.sch (KiCad schematic (older format))
At the start: 54 parts, among them J1 USB_B_Micro, J2 AudioJack4, SW1 SW_PUSH, SW10 SW_PUSH, SW11 SW_PUSH, SW12 SW_PUSH, SW13 SW_PUSH, SW14 SW_PUSH, SW15 SW_PUSH, SW16 SW_PUSH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

Commit message: Done with routing
Connections:
- net col0: now also U1.15 (PB1); no longer U1.10 (PD4)
- net col1: now also U1.16 (PB2); no longer U1.11 (PD5)
- net col2: now also U1.17 (PB3); no longer U1.12 (PD6)
- net col3: now also U1.18 (PB4); no longer U1.14 (PB0)
- net col4: now also U1.19 (PB5); no longer U1.15 (PB1)
- net col5: now also U1.20 (PB6); no longer U1.16 (PB2)
- net col6: now also U1.21 (PB7); no longer U1.9 (PD3)
- net data: now also U1.23 (PC6); no longer U1.8 (PD2)
- net row1: now also U1.14 (PB0); no longer U1.25 (PC5)
- net row2: now also U1.22 (PC7); no longer U1.23 (PC6)
Changed lines of the file:
@@
 Wire Wire Line
 	9275 925  9275 2550
-Text GLabel 6225 5925 2    50   Input Italic 0
+Text GLabel 6225 4825 2    50   Input Italic 0
 col6
 Text Notes 3175 3175 2    50   Italic 0
@@
 Wire Wire Line
 	2900 3575 2900 3475
-Text GLabel 6225 5825 2    50   Input Italic 0
+Text GLabel 6225 5325 2    50   Input Italic 0
 data
 $Comp
@@
 Text GLabel 6225 5125 2    50   Input Italic 0
 row0
-Text GLabel 6225 5225 2    50   Input Italic 0
+Text GLabel 6225 4125 2    50   Input Italic 0
 row1
-Text GLabel 6225 5325 2    50   Input Italic 0
+Text GLabel 6225 5425 2    50   Input Italic 0
 row2
-Text GLabel 6225 6025 2    50   Input Italic 0
+Text GLabel 6225 4225 2    50   Input Italic 0
 col0
-Text GLabel 6225 6125 2    50   Input Italic 0
+Text GLabel 6225 4325 2    50   Input Italic 0
 col1
-Text GLabel 6225 6225 2    50   Input Italic 0
+Text GLabel 6225 4425 2    50   Input Italic 0
 col2
-Text GLabel 6225 4125 2    50   Input Italic 0
+Text GLabel 6225 4525 2    50   Input Italic 0
 col3
-Text GLabel 6225 4225 2    50   Input Italic 0
+Text GLabel 6225 4625 2    50   Input Italic 0
 col4
-Text GLabel 6225 4325 2    50   Input Italic 0
+Text GLabel 6225 4725 2    50   Input Italic 0
 col5
 $Comp
@@
 	6125 5125 6225 5125
 Wire Wire Line
-	6125 5225 6225 5225
-Wire Wire Line
-	6125 5325 6225 5325
-Wire Wire Line
 	4575 4125 4725 4125
-NoConn ~ 6125 5425
 NoConn ~ 6125 5625
 $Comp
@@
 Wire Wire Line
 	950  6600 950  6800
-NoConn ~ 6125 4625
 $Comp
 L Device:R_Small R4
@@
 Wire Wire Line
 	6200 6600 6200 6650
-Wire Wire Line
-	6125 4325 6225 4325
-Wire Wire Line
-	6125 4225 6225 4225
-Wire Wire Line
-	6125 4125 6225 4125
-Wire Wire Line
-	6125 6225 6225 6225
-Wire Wire Line
-	6125 6025 6225 6025
-Wire Wire Line
-	6125 6125 6225 6125
-NoConn ~ 6125 4425
-NoConn ~ 6125 4525
-NoConn ~ 6125 4725
-NoConn ~ 6125 4825
 NoConn ~ 6125 5025
 NoConn ~ 6125 5725
-Wire Wire Line
-	6125 5925 6225 5925
-Wire Wire Line
-	6125 5825 6225 5825
 Text GLabel 8400 925  1    50   Input Italic 0
 col5
@@
 	1    0    0    -1
 $EndComp
+Wire Wire Line
+	6125 5325 6225 5325
+Wire Wire Line
+	6125 5425 6225 5425
+NoConn ~ 6125 5825
+Wire Wire Line
+	6125 4825 6225 4825
+NoConn ~ 6125 5925
+Wire Wire Line
+	6125 4725 6225 4725
+Wire Wire Line
+	6125 4625 6225 4625
+Wire Wire Line
+	6125 4525 6225 4525
+Wire Wire Line
+	6125 4425 6225 4425
+NoConn ~ 6125 6225
+Wire Wire Line
+	6125 4325 6225 4325
+NoConn ~ 6125 6125
+NoConn ~ 6125 6025
+Wire Wire Line
+	6125 4225 6225 4225
+Wire Wire Line
+	6125 4125 6225 4125
+NoConn ~ 6125 5225
 $EndSCHEMATC

Commit message: PCB almost there...
Parts:
- added RR1: 10k, Resistor_SMD:R_0805_2012Metric_Pad1.20x1.40mm_HandSolder, symbol Device:R_Small
Connections:
- net GND: now also RR1.2
- net data: now also U1.8 (PD2); no longer U1.23 (PC6)
- net at U1.12 (PD6): now also RR1.1
- no-connect marks 11 -> 10
Other:
- note added: "NOTE:\n1. data (serial to other hand) needs to be connected to INT*:\nD0,D1,D2,D3, (probably C7,D4,D6 too?)\n\n2. HWB (D7) need to be grounded through pull-down resistor\nto force start from boot loader.\n\n3. PD6 is reserved and is connected to pull-down resistor\nso if split-hand indicator EEPROM is not working then\nthis pin is to indicate whether this is master or slave.\n\n4. Other GPIO pins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"
Changed lines of the file:
@@
 Wire Wire Line
 	2900 3575 2900 3475
-Text GLabel 6225 5325 2    50   Input Italic 0
+Text GLabel 6225 5825 2    50   Input Italic 0
 data
 $Comp
@@
 $EndComp
 Wire Wire Line
-	6125 5325 6225 5325
-Wire Wire Line
 	6125 5425 6225 5425
-NoConn ~ 6125 5825
 Wire Wire Line
 	6125 4825 6225 4825
@@
 Wire Wire Line
 	6125 4425 6225 4425
-NoConn ~ 6125 6225
 Wire Wire Line
 	6125 4325 6225 4325
@@
 	6125 4125 6225 4125
 NoConn ~ 6125 5225
+Text Notes 6950 4850 0    50   ~ 0
+NOTE:\n1. data (serial to other hand) needs to be connected to INT*:\nD0,D1,D2,D3, (probably C7,D4,D6 too?)\n\n2. HWB (D7) need to be grounded through pull-down resistor\nto force start from boot loader.\n\n3. PD6 is reserved and is connected to pull-down resistor\nso if split-hand indicator EEPROM is not working then\nthis pin is to indicate whether this is master or slave.\n\n4. Other GPIO pins (row*, col*) are selected to simplify routing on PCB.
+Wire Wire Line
+	6125 5825 6225 5825
+NoConn ~ 6125 5325
+$Comp
+L Device:R_Small RR1
+U 1 1 600CEBFB
+P 6500 6500
+F 0 "RR1" H 6559 6546 50  0000 L CNN
+F 1 "10k" H 6559 6455 50  0000 L CNN
+F 2 "Resistor_SMD:R_0805_2012Metric_Pad1.20x1.40mm_HandSolder" H 6500 6500 50  0001 C CNN
+F 3 "~" H 6500 6500 50  0001 C CNN
+	1    6500 6500
+	1    0    0    -1
+$EndComp
+$Comp
+L power:GND #PWR?
+U 1 1 600CF505
+P 6500 6650
+F 0 "#PWR?" H 6500 6400 50  0001 C CNN
+F 1 "GND" H 6505 6477 50  0000 C CNN
+F 2 "" H 6500 6650 50  0001 C CNN
+F 3 "" H 6500 6650 50  0001 C CNN
+	1    6500 6650
+	1    0    0    -1
+$EndComp
+Wire Wire Line
+	6500 6600 6500 6650
+Wire Wire Line
+	6125 6225 6500 6225
+Wire Wire Line
+	6500 6225 6500 6400
 $EndSCHEMATC

Commit message: pisces V2.1 option 2 (SPLIT_HAND_MATRIX_GRID)
Parts:
- removed RR1: 10k, Resistor_SMD:R_0805_2012Metric_Pad1.20x1.40mm_HandSolder, symbol Device:R_Small
- added D_H1: D, kbd:D3_SMD, symbol Device:D
- added R5: 10k, Resistor_SMD:R_0805_2012Metric_Pad1.20x1.40mm_HandSolder, symbol Device:R_Small
Connections:
- net GND: now also R5.2
- net col6: now also D_H1.2 (A)
- net data: now also R5.1
- net row1: now also D_H1.1 (K)
- no-connect marks 10 -> 11
Other:
- note added: "NOTE:\n1. data (serial to other hand) needs to be connected to INT*:\nD0,D1,D2,D3, (probably C7,D4,D6 too?)\n\n2. HWB (D7) need to be grounded through pull-down resistor\nto force start from boot loader.\n\n3. Other GPIO pins (row*, col*) are selected to simplify routing on PCB."
- note removed: "NOTE:\n1. data (serial to other hand) needs to be connected to INT*:\nD0,D1,D2,D3, (probably C7,D4,D6 too?)\n\n2. HWB (D7) need to be grounded through pull-down resistor\nto force start from boot loader.\n\n3. PD6 is reserved and is connected to pull-down resistor\nso if split-hand indicator EEPROM is not working then\nthis pin is to indicate whether this is master or slave.\n\n4. Other GPIO pins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"
Changed lines of the file:
@@
 col6
 Wire Wire Line
-	9275 925  9275 2550
+	9275 925  9275 1925
 Text GLabel 6225 4825 2    50   Input Italic 0
 col6
@@
 Wire Wire Line
 	2650 3775 2900 3775
-Text GLabel 2900 3475 2    50   Input Italic 0
+Text GLabel 3250 3575 2    50   Input Italic 0
 data
-Wire Wire Line
-	2650 3575 2900 3575
-Wire Wire Line
-	2900 3575 2900 3475
 Text GLabel 6225 5825 2    50   Input Italic 0
 data
@@
 NoConn ~ 6125 5225
 Text Notes 6950 4850 0    50   ~ 0
-NOTE:\n1. data (serial to other hand) needs to be connected to INT*:\nD0,D1,D2,D3, (probably C7,D4,D6 too?)\n\n2. HWB (D7) need to be grounded through pull-down resistor\nto force start from boot loader.\n\n3. PD6 is reserved and is connected to pull-down resistor\nso if split-hand indicator EEPROM is not working then\nthis pin is to indicate whether this is master or slave.\n\n4. Other GPIO pins (row*, col*) are selected to simplify routing on PCB.
+NOTE:\n1. data (serial to other hand) needs to be connected to INT*:\nD0,D1,D2,D3, (probably C7,D4,D6 too?)\n\n2. HWB (D7) need to be grounded through pull-down resistor\nto force start from boot loader.\n\n3. Other GPIO pins (row*, col*) are selected to simplify routing on PCB.
 Wire Wire Line
 	6125 5825 6225 5825
 NoConn ~ 6125 5325
 $Comp
-L Device:R_Small RR1
-U 1 1 600CEBFB
-P 6500 6500
-F 0 "RR1" H 6559 6546 50  0000 L CNN
-F 1 "10k" H 6559 6455 50  0000 L CNN
-F 2 "Resistor_SMD:R_0805_2012Metric_Pad1.20x1.40mm_HandSolder" H 6500 6500 50  0001 C CNN
-F 3 "~" H 6500 6500 50  0001 C CNN
-	1    6500 6500
-	1    0    0    -1
-$EndComp
-$Comp
-L power:GND #PWR?
-U 1 1 600CF505
-P 6500 6650
-F 0 "#PWR?" H 6500 6400 50  0001 C CNN
-F 1 "GND" H 6505 6477 50  0000 C CNN
-F 2 "" H 6500 6650 50  0001 C CNN
-F 3 "" H 6500 6650 50  0001 C CNN
-	1    6500 6650
-	1    0    0    -1
-$EndComp
-Wire Wire Line
-	6500 6600 6500 6650
-Wire Wire Line
-	6125 6225 6500 6225
-Wire Wire Line
-	6500 6225 6500 6400
+L Device:D D_H1
+U 1 1 603BE437
+P 9875 2075
+F 0 "D_H1" V 9921 1995 50  0000 R CNN
+F 1 "D" V 9830 1995 50  0000 R CNN
+F 2 "kbd:D3_SMD" H 9875 2075 50  0001 C CNN
+F 3 "~" H 9875 2075 50  0001 C CNN
+	1    9875 2075
+	0    -1   -1   0
+$EndComp
+Wire Wire Line
+	9000 2225 9875 2225
+Connection ~ 9000 2225
+Wire Wire Line
+	9875 1925 9275 1925
+Connection ~ 9275 1925
+Wire Wire Line
+	9275 1925 9275 2550
+Wire Wire Line
+	2650 3575 3150 3575
+$Comp
+L power:GND #PWR0108
+U 1 1 603CFDA7
+P 3150 3900
+F 0 "#PWR0108" H 3150 3650 50  0001 C CNN
+F 1 "GND" H 3155 3727 50  0000 C CNN
+F 2 "" H 3150 3900 50  0001 C CNN
+F 3 "" H 3150 3900 50  0001 C CNN
+	1    3150 3900
+	1    0    0    -1
+$EndComp
+$Comp
+L Device:R_Small R5
+U 1 1 603D0C12
+P 3150 3750
+F 0 "R5" H 3209 3796 50  0000 L CNN
+F 1 "10k" H 3209 3705 50  0000 L CNN
+F 2 "Resistor_SMD:R_0805_2012Metric_Pad1.20x1.40mm_HandSolder" H 3150 3750 50  0001 C CNN
+F 3 "~" H 3150 3750 50  0001 C CNN
+	1    3150 3750
+	1    0    0    -1
+$EndComp
+Wire Wire Line
+	3150 3900 3150 3850
+Wire Wire Line
+	3150 3650 3150 3575
+Connection ~ 3150 3575
+Wire Wire Line
+	3150 3575 3250 3575
+NoConn ~ 6125 6225
 $EndSCHEMATC

Commit message: Regenerated pisces pcb gerber files
Other:
- note added: "NOTE:\nD_H1 is used for handness.\n(SPLIT_HAND_MATRIX_GRID).\nNeed to implement only one hand."
- note added: "NOTE:\nR5 is for \nterminate resistor"
Changed lines of the file:
@@
 	3150 3575 3250 3575
 NoConn ~ 6125 6225
+Text Notes 3400 3900 0    50   ~ 0
+NOTE:\nR5 is for \nterminate resistor
+Text Notes 9825 1875 0    50   ~ 0
+NOTE:\nD_H1 is used for handness.\n(SPLIT_HAND_MATRIX_GRID).\nNeed to implement only one hand.
 $EndSCHEMATC

Commit message: Verified that the current drawing is okay on KiCad 5.1.12 (#29)
Parts:
- C1, C2, C4, C5, C6: symbol Device:C_Small -> pisces-rescue:C_Small-Device
- C3: symbol Device:C -> pisces-rescue:C-Device
- D1, D10, D11, D12, D13, D14, D15, D16, D17, D18, D19, D2, D3, D4, D5, D6, D7, D8, D9, D_H1: symbol Device:D -> pisces-rescue:D-Device
- F1: symbol Device:Polyfuse_Small -> pisces-rescue:Polyfuse_Small-Device
- J1: symbol Connector:USB_B_Micro -> pisces-rescue:USB_B_Micro-Connector
- J2: symbol Connector:AudioJack4 -> pisces-rescue:AudioJack4-Connector
- R1, R2, R3: symbol Device:R -> pisces-rescue:R-Device
- R4, R5: symbol Device:R_Small -> pisces-rescue:R_Small-Device
- RSTSW1, SW1, SW10, SW11, SW12, SW13, SW14, SW15, SW16, SW17, SW18, SW19, SW2, SW3, SW4, SW5, SW6, SW7, SW8, SW9: symbol kbd:SW_PUSH -> pisces-rescue:SW_PUSH-kbd
- U1: symbol MCU_Microchip_ATmega:ATmega32U2-AU -> pisces-rescue:ATmega32U2-AU-MCU_Microchip_ATmega
- Y1: symbol Device:Crystal_GND24_Small -> pisces-rescue:Crystal_GND24_Small-Device

Commit message: Removed R5 (resistor) from schematic (#30)
Parts:
- removed R5: 10k, Resistor_SMD:R_0805_2012Metric_Pad1.20x1.40mm_HandSolder, symbol pisces-rescue:R_Small-Device
Other:
- note removed: "NOTE:\nR5 is for \nterminate resistor"
Changed lines of the file:
@@
 Wire Wire Line
 	9275 1925 9275 2550
-Wire Wire Line
-	2650 3575 3150 3575
-$Comp
-L pisces-rescue:GND-power #PWR0108
-U 1 1 603CFDA7
-P 3150 3900
-F 0 "#PWR0108" H 3150 3650 50  0001 C CNN
-F 1 "GND" H 3155 3727 50  0000 C CNN
-F 2 "" H 3150 3900 50  0001 C CNN
-F 3 "" H 3150 3900 50  0001 C CNN
-	1    3150 3900
-	1    0    0    -1
-$EndComp
-$Comp
-L pisces-rescue:R_Small-Device R5
-U 1 1 603D0C12
-P 3150 3750
-F 0 "R5" H 3209 3796 50  0000 L CNN
-F 1 "10k" H 3209 3705 50  0000 L CNN
-F 2 "Resistor_SMD:R_0805_2012Metric_Pad1.20x1.40mm_HandSolder" H 3150 3750 50  0001 C CNN
-F 3 "~" H 3150 3750 50  0001 C CNN
-	1    3150 3750
-	1    0    0    -1
-$EndComp
-Wire Wire Line
-	3150 3900 3150 3850
-Wire Wire Line
-	3150 3650 3150 3575
-Connection ~ 3150 3575
-Wire Wire Line
-	3150 3575 3250 3575
 NoConn ~ 6125 6225
-Text Notes 3400 3900 0    50   ~ 0
-NOTE:\nR5 is for \nterminate resistor
 Text Notes 9825 1875 0    50   ~ 0
 NOTE:\nD_H1 is used for handness.\n(SPLIT_HAND_MATRIX_GRID).\nNeed to implement only one hand.
+Wire Wire Line
+	2650 3575 3250 3575
 $EndSCHEMATC

Commit message: Stopped using hand-soldering footprint for most of parts
Parts:
- C1, C2, C3, C5, C6: footprint Capacitor_SMD:C_0603_1608Metric_Pad1.08x0.95mm_HandSolder -> Capacitor_SMD:C_0603_1608Metric
- C4: footprint Capacitor_SMD:C_0805_2012Metric_Pad1.18x1.45mm_HandSolder -> Capacitor_SMD:C_0805_2012Metric
- R1, R2, R3, R4: footprint Resistor_SMD:R_0805_2012Metric_Pad1.20x1.40mm_HandSolder -> Resistor_SMD:R_0805_2012Metric
- Y1: footprint Crystal:Crystal_SMD_SeikoEpson_FA238-4Pin_3.2x2.5mm_HandSoldering -> Crystal:Crystal_SMD_SeikoEpson_FA238-4Pin_3.2x2.5mm
Changed lines of the file:
@@
 F 0 "R1" V 1293 6200 50  0000 C CNN
 F 1 "22" V 1384 6200 50  0000 C CNN
-F 2 "Resistor_SMD:R_0805_2012Metric_Pad1.20x1.40mm_HandSolder" V 1430 6200 50  0001 C CNN
+F 2 "Resistor_SMD:R_0805_2012Metric" V 1430 6200 50  0001 C CNN
 F 3 "~" H 1500 6200 50  0001 C CNN
 	1    1500 6200
@@
 F 0 "R2" V 1543 6300 50  0000 C CNN
 F 1 "22" V 1634 6300 50  0000 C CNN
-F 2 "Resistor_SMD:R_0805_2012Metric_Pad1.20x1.40mm_HandSolder" V 1680 6300 50  0001 C CNN
+F 2 "Resistor_SMD:R_0805_2012Metric" V 1680 6300 50  0001 C CNN
 F 3 "~" H 1750 6300 50  0001 C CNN
 	1    1750 6300
@@
 F 0 "R3" H 4645 3921 50  0000 L CNN
 F 1 "10k" H 4645 3830 50  0000 L CNN
-F 2 "Resistor_SMD:R_0805_2012Metric_Pad1.20x1.40mm_HandSolder" V 4505 3875 50  0001 C CNN
+F 2 "Resistor_SMD:R_0805_2012Metric" V 4505 3875 50  0001 C CNN
 F 3 "~" H 4575 3875 50  0001 C CNN
 	1    4575 3875
@@
 F 0 "C3" H 4715 5221 50  0000 L CNN
 F 1 "0.1u" H 4715 5130 50  0000 L CNN
-F 2 "Capacitor_SMD:C_0603_1608Metric_Pad1.08x0.95mm_HandSolder" H 4638 5025 50  0001 C CNN
+F 2 "Capacitor_SMD:C_0603_1608Metric" H 4638 5025 50  0001 C CNN
 F 3 "~" H 4600 5175 50  0001 C CNN
 	1    4600 5175
@@
 F 0 "Y1" V 4054 4569 50  0000 L CNN
 F 1 "Crystal_GND24_Small" V 4145 4569 50  0000 L CNN
-F 2 "Crystal:Crystal_SMD_SeikoEpson_FA238-4Pin_3.2x2.5mm_HandSoldering" H 4100 4425 50  0001 C CNN
+F 2 "Crystal:Crystal_SMD_SeikoEpson_FA238-4Pin_3.2x2.5mm" H 4100 4425 50  0001 C CNN
 F 3 "~" H 4100 4425 50  0001 C CNN
 	1    4100 4425
@@
 F 0 "C1" H 3692 4496 50  0000 L CNN
 F 1 "22p" H 3692 4405 50  0000 L CNN
-F 2 "Capacitor_SMD:C_0603_1608Metric_Pad1.08x0.95mm_HandSolder" H 3600 4450 50  0001 C CNN
+F 2 "Capacitor_SMD:C_0603_1608Metric" H 3600 4450 50  0001 C CNN
 F 3 "~" H 3600 4450 50  0001 C CNN
 	1    3600 4450
@@
 F 0 "C2" H 3867 4671 50  0000 L CNN
 F 1 "22p" H 3867 4580 50  0000 L CNN
-F 2 "Capacitor_SMD:C_0603_1608Metric_Pad1.08x0.95mm_HandSolder" H 3775 4625 50  0001 C CNN
+F 2 "Capacitor_SMD:C_0603_1608Metric" H 3775 4625 50  0001 C CNN
 F 3 "~" H 3775 4625 50  0001 C CNN
 	1    3775 4625
@@
 F 0 "C4" H 2592 6146 50  0000 L CNN
 F 1 "10u" H 2592 6055 50  0000 L CNN
-F 2 "Capacitor_SMD:C_0805_2012Metric_Pad1.18x1.45mm_HandSolder" H 2500 6100 50  0001 C CNN
+F 2 "Capacitor_SMD:C_0805_2012Metric" H 2500 6100 50  0001 C CNN
 F 3 "~" H 2500 6100 50  0001 C CNN
 	1    2500 6100
@@
 F 0 "C5" H 2892 6146 50  0000 L CNN
 F 1 "1u" H 2892 6055 50  0000 L CNN
-F 2 "Capacitor_SMD:C_0603_1608Metric_Pad1.08x0.95mm_HandSolder" H 2800 6100 50  0001 C CNN
+F 2 "Capacitor_SMD:C_0603_1608Metric" H 2800 6100 50  0001 C CNN
 F 3 "~" H 2800 6100 50  0001 C CNN
 	1    2800 6100
@@
 F 0 "C6" H 3192 6146 50  0000 L CNN
 F 1 "0.1u" H 3192 6055 50  0000 L CNN
-F 2 "Capacitor_SMD:C_0603_1608Metric_Pad1.08x0.95mm_HandSolder" H 3100 6100 50  0001 C CNN
+F 2 "Capacitor_SMD:C_0603_1608Metric" H 3100 6100 50  0001 C CNN
 F 3 "~" H 3100 6100 50  0001 C CNN
 	1    3100 6100
@@
 F 0 "R4" H 6259 6546 50  0000 L CNN
 F 1 "10k" H 6259 6455 50  0000 L CNN
-F 2 "Resistor_SMD:R_0805_2012Metric_Pad1.20x1.40mm_HandSolder" H 6200 6500 50  0001 C CNN
+F 2 "Resistor_SMD:R_0805_2012Metric" H 6200 6500 50  0001 C CNN
 F 3 "~" H 6200 6500 50  0001 C CNN
 	1    6200 6500

Commit message: Used smaller parts footprint (Resistors and Capacitors) (#32)
* Resistors: 0805 --> 0603, Capacitors (other than 10u): 0603

* Smaller parts footprint
Parts:
- C1, C2, C3, C6: footprint Capacitor_SMD:C_0603_1608Metric -> Capacitor_SMD:C_0402_1005Metric
- R1, R2, R3, R4: footprint Resistor_SMD:R_0805_2012Metric -> Resistor_SMD:R_0603_1608Metric
Changed lines of the file:
@@
 F 0 "R1" V 1293 6200 50  0000 C CNN
 F 1 "22" V 1384 6200 50  0000 C CNN
-F 2 "Resistor_SMD:R_0805_2012Metric" V 1430 6200 50  0001 C CNN
+F 2 "Resistor_SMD:R_0603_1608Metric" V 1430 6200 50  0001 C CNN
 F 3 "~" H 1500 6200 50  0001 C CNN
 	1    1500 6200
@@
 F 0 "R2" V 1543 6300 50  0000 C CNN
 F 1 "22" V 1634 6300 50  0000 C CNN
-F 2 "Resistor_SMD:R_0805_2012Metric" V 1680 6300 50  0001 C CNN
+F 2 "Resistor_SMD:R_0603_1608Metric" V 1680 6300 50  0001 C CNN
 F 3 "~" H 1750 6300 50  0001 C CNN
 	1    1750 6300
@@
 F 0 "R3" H 4645 3921 50  0000 L CNN
 F 1 "10k" H 4645 3830 50  0000 L CNN
-F 2 "Resistor_SMD:R_0805_2012Metric" V 4505 3875 50  0001 C CNN
+F 2 "Resistor_SMD:R_0603_1608Metric" V 4505 3875 50  0001 C CNN
 F 3 "~" H 4575 3875 50  0001 C CNN
 	1    4575 3875
@@
 F 0 "C3" H 4715 5221 50  0000 L CNN
 F 1 "0.1u" H 4715 5130 50  0000 L CNN
-F 2 "Capacitor_SMD:C_0603_1608Metric" H 4638 5025 50  0001 C CNN
+F 2 "Capacitor_SMD:C_0402_1005Metric" H 4638 5025 50  0001 C CNN
 F 3 "~" H 4600 5175 50  0001 C CNN
 	1    4600 5175
@@
 F 0 "C1" H 3692 4496 50  0000 L CNN
 F 1 "22p" H 3692 4405 50  0000 L CNN
-F 2 "Capacitor_SMD:C_0603_1608Metric" H 3600 4450 50  0001 C CNN
+F 2 "Capacitor_SMD:C_0402_1005Metric" H 3600 4450 50  0001 C CNN
 F 3 "~" H 3600 4450 50  0001 C CNN
 	1    3600 4450
@@
 F 0 "C2" H 3867 4671 50  0000 L CNN
 F 1 "22p" H 3867 4580 50  0000 L CNN
-F 2 "Capacitor_SMD:C_0603_1608Metric" H 3775 4625 50  0001 C CNN
+F 2 "Capacitor_SMD:C_0402_1005Metric" H 3775 4625 50  0001 C CNN
 F 3 "~" H 3775 4625 50  0001 C CNN
 	1    3775 4625
@@
 F 0 "C6" H 3192 6146 50  0000 L CNN
 F 1 "0.1u" H 3192 6055 50  0000 L CNN
-F 2 "Capacitor_SMD:C_0603_1608Metric" H 3100 6100 50  0001 C CNN
+F 2 "Capacitor_SMD:C_0402_1005Metric" H 3100 6100 50  0001 C CNN
 F 3 "~" H 3100 6100 50  0001 C CNN
 	1    3100 6100
@@
 F 0 "R4" H 6259 6546 50  0000 L CNN
 F 1 "10k" H 6259 6455 50  0000 L CNN
-F 2 "Resistor_SMD:R_0805_2012Metric" H 6200 6500 50  0001 C CNN
+F 2 "Resistor_SMD:R_0603_1608Metric" H 6200 6500 50  0001 C CNN
 F 3 "~" H 6200 6500 50  0001 C CNN
 	1    6200 6500
